File: hardware/MeshangerV/MeshangerV.sch (KiCad schematic (older format))
At the start: 11 parts

Commit message: more schmatic work
Parts:
- removed C? (x2): C_Small, symbol Device:C_Small
- removed R?: R_Small, symbol Device:R_Small
- removed SW?: SW_Push, symbol Switch:SW_Push
- removed U?: CH554G, symbol MCU_WCH:CH554G
- added BT?: Battery_Cell, symbol Device:Battery_Cell
- added C? (x18): C_Small, symbol Device:C_Small
- added D? (x3): D_Schottky, symbol Device:D_Schottky
- added L? (x2): L_Small, symbol Device:L_Small
- added R? (x9): R_Small, symbol Device:R_Small
- added U?: ESP32-C3, Package_DFN_QFN:QFN-32-1EP_5x5mm_P0.5mm_EP3.45x3.45mm, symbol MCU_Espressif:ESP32-C3
- added U?: AP3012KTR-G1, symbol Diodes_inc:AP3012KTR-G1
- added U?: AP7333-33SRG-7, TO_SOT_Packages_SMD:SOT-23, symbol Diodes_inc:AP7333-33SRG-7
- added Y?: 32k, symbol Device:Crystal
- added Y?: 40MHz, symbol Device:Crystal
Connections:
- net labels added: +3.3VA, ANT, BAT_SHDN, BVOLT, CHRG_EN, VDDA, V_BAT, _CHRG
- net labels removed: -CHRG, ESP_ENABLE, ESP_INT, USBRX, USBTX, bload, vbat
- wire segments 67 -> 176
Other:
- note removed: "bootsequece -> ch554 -> is off or charging ->esp enable ->recieve usb sd for writing-> ch554 device shutdown"
- moved on the sheet: C?, R?, U?

Commit message: more schematic
Parts:
- J?: symbol Connector:USB_C_Receptacle_USB2.0 -> MeshangerV-rescue:USB_C_Receptacle_USB2.0-Connector
- U?: symbol MCU_Espressif:ESP32-C3 -> MeshangerV-rescue:ESP32-C3-MCU_Espressif
- U?: symbol BATMAN_TopPower:TP4056 -> MeshangerV-rescue:TP4056-BATMAN_TopPower
- U?: symbol Diodes_inc:AP3012KTR-G1 -> MeshangerV-rescue:AP3012KTR-G1-Diodes_inc
Changed lines of the file:
@@
 EESchema Schematic File Version 4
 LIBS:MeshangerV-cache
-EELAYER 29 0
+EELAYER 26 0
 EELAYER END
 $Descr A4 11693 8268
 encoding utf-8
-Sheet 1 3
+Sheet 1 4
 Title ""
 Date ""
@@
 $EndComp
 $Comp
-L Connector:USB_C_Receptacle_USB2.0 J?
+L MeshangerV-rescue:USB_C_Receptacle_USB2.0-Connector J?
 U 1 1 5FBDAB30
 P 1200 2600
@@
 	5350 3250 5650 3250
 $Comp
-L BATMAN_TopPower:TP4056 U?
+L MeshangerV-rescue:TP4056-BATMAN_TopPower U?
 U 1 1 5FBEC96F
 P 2100 6300
@@
 	2550 6400 3000 6400
 $Comp
-L MCU_Espressif:ESP32-C3 U?
+L MeshangerV-rescue:ESP32-C3-MCU_Espressif U?
 U 1 1 5FBE8965
 P 9700 3700
@@
 V_BAT
 $Comp
-L Diodes_inc:AP3012KTR-G1 U?
+L MeshangerV-rescue:AP3012KTR-G1-Diodes_inc U?
 U 1 1 5FC8278B
 P 5650 6700
@@
 	1200 3750 1200 3900
 $Sheet
-S 7700 650  1900 1100
+S 9050 600  1350 750
 U 5FDFC263
 F0 "Display hardware" 50
 F1 "display.sch" 50
+F2 "3V3" I L 9050 700 50
+F3 "GND" I L 9050 1250 50
+F4 "LCD_CS" I R 10400 700 50
+F5 "LCD_SCLK" I R 10400 800 50
+F6 "LCD_MOSI" I R 10400 900 50
+F7 "LCD_DC" I R 10400 1000 50
 $EndSheet
 $Sheet
@@
 F8 "LED_SD" I R 7150 1250 50
 $EndSheet
+$Sheet
+S 5600 1550 1500 800
+U 5FC5BE78
+F0 "antenna" 50
+F1 "antenna.sch" 50
+$EndSheet
 $EndSCHEMATC

Commit message: schematic complete more or less
Parts:
- removed D?: D_Schottky, symbol Device:D_Schottky
- removed R?: R_Small, symbol Device:R_Small
- added C? (x2): C_Small, symbol Device:C_Small
- added C?: CP, symbol Device:CP
- added J?: Conn_01x20_Male, symbol Connector:Conn_01x20_Male
- added JP? (x2): SolderJumper_3_Bridged12, symbol Jumper:SolderJumper_3_Bridged12
- added R? (x2): R_Small, symbol Device:R_Small
- added RN?: R_Pack04, symbol Device:R_Pack04
Connections:
- net labels added: BLSEL, CHRG_SD, CHUSB+, CHUSB-, ESPUSB+, ESPUSB-, ESP_ENABLE, ESP_RESET, ESP_RX, ESP_TX, INPUTINT, LCD_BL_EN, LCD_CS, LCD_DC, LED_SD, MISO, MOSI, SCK, SCL, SDA, SPICS0, SPID, SPIHD, SPIQ, SPISCK, SPIWP, SPI_VCC
- net labels removed: CHRG_EN, USB+, USB-, VDDA
- wire segments 176 -> 293
Other:
- note added: "BLSEL 1 = SPI 0=DOWNLOAD"
- note added: "BOOT STRAPPING GPIO HIGH PREVENTS UNWANTED MODE"
- note added: "Bulk caps to allow battery to take over"
- note removed: "needs 5v to program\n"
- moved on the sheet: D?, J?, L?, R?

Commit message: routing has begun
Parts:
- BT1: renamed from BT?; footprint (none) -> Connectors_JST:JST_PH_S2B-PH-SM4-TB_02x2.00mm_Angled
- C1, C11, C12, C13, C16, C18, C19, C2, C20, C21, C22, C23, C4, C5, C6, C7, C9: renamed from C?; footprint (none) -> Capacitor_SMD:C_0603_1608Metric
- C10, C8: renamed from C?; value C_Small -> 1uF; footprint (none) -> Capacitor_SMD:C_0603_1608Metric
- C14, C15: renamed from C?; value C_Small -> 22uF; footprint (none) -> Capacitor_SMD:C_0805_2012Metric
- C17: renamed from C?; value C_Small -> 10uF; footprint (none) -> Capacitor_SMD:C_0805_2012Metric
- C3: renamed from C?; footprint (none) -> Capacitor_SMD:CP_Elec_4x4.5
- D1, D2: renamed from D?; footprint (none) -> Diode_SMD:D_SOD-323
- J1: renamed from J?; footprint (none) -> footprint:VACON_CSP_USC16_TR
- J2: renamed from J?; footprint (none) -> Connector_PinSocket_2.54mm:PinSocket_1x20_P2.54mm_Vertical
- JP1, JP2: renamed from JP?; footprint (none) -> Jumper:SolderJumper-3_P1.3mm_Bridged12_RoundedPad1.0x1.5mm
- L1: renamed from L?; footprint (none) -> Inductors_SMD:L_1210
- L2: renamed from L?; footprint (none) -> Inductors_SMD:L_Taiyo-Yuden_NR-40xx_HandSoldering
- R1, R10, R11, R2, R3, R4, R5, R6, R7, R8, R9: renamed from R?; footprint (none) -> Resistor_SMD:R_0603_1608Metric
- RN1: renamed from RN?; footprint (none) -> Resistor_SMD:R_Array_Convex_4x0603
- U1: renamed from U?; footprint (none) -> Package_SO:SOIC-8-1EP_3.9x4.9mm_P1.27mm_EP2.35x2.35mm
- U4: renamed from U?; footprint (none) -> Package_TO_SOT_SMD:SOT-23-5
- Y1: renamed from Y?; footprint (none) -> Crystal:Crystal_SMD_Abracon_ABM8G-4Pin_3.2x2.5mm
- Y2: renamed from Y?; footprint (none) -> Crystal:Crystal_AT310_D3.0mm_L10.0mm_Horizontal
- gave numbers to parts that had none: 3
