File: hardware/MeshangerV/debug.sch (KiCad schematic (older format))
At the start: 4 parts

Commit message: routing has begun
Parts:
- D12: renamed from D?; footprint (none) -> Diode_SMD:D_SOD-323
- TP10, TP11: renamed from TP?; footprint (none) -> TestPoint:TestPoint_Pad_1.5x1.5mm
- U9: renamed from U?; footprint (none) -> Package_SO:SOIC-16_3.9x9.9mm_P1.27mm; symbol MCU_WCH:CH552G -> MeshangerV-rescue:CH552G-MCU_WCH
Changed lines of the file:
@@
 EESchema Schematic File Version 4
 LIBS:MeshangerV-cache
-EELAYER 29 0
+EELAYER 26 0
 EELAYER END
 $Descr A4 11693 8268
@@
 3V3
 $Comp
-L MCU_WCH:CH552G U?
+L MeshangerV-rescue:CH552G-MCU_WCH U9
 U 1 1 5FDED1AF
 P 7200 3600
-F 0 "U?" H 7175 4315 50  0000 C CNN
+F 0 "U9" H 7175 4315 50  0000 C CNN
 F 1 "CH552G" H 7175 4224 50  0000 C CNN
-F 2 "" H 7500 3600 50  0001 C CNN
+F 2 "Package_SO:SOIC-16_3.9x9.9mm_P1.27mm" H 7500 3600 50  0001 C CNN
 F 3 "" H 7500 3600 50  0001 C CNN
 	1    7200 3600
@@
 P 2200 600
 AR Path="/5FDEDEFB" Ref="#PWR?"  Part="1"
-AR Path="/5FDE49AF/5FDEDEFB" Ref="#PWR?"  Part="1"
-F 0 "#PWR?" H 2200 450 50  0001 C CNN
+AR Path="/5FDE49AF/5FDEDEFB" Ref="#PWR0169"  Part="1"
+F 0 "#PWR0169" H 2200 450 50  0001 C CNN
 F 1 "VBUS" H 2215 773 50  0000 C CNN
 F 2 "" H 2200 600 50  0001 C CNN
@@
 P 5500 2800
 AR Path="/5FDF0272" Ref="#PWR?"  Part="1"
-AR Path="/5FDE49AF/5FDF0272" Ref="#PWR?"  Part="1"
-F 0 "#PWR?" H 5500 2650 50  0001 C CNN
+AR Path="/5FDE49AF/5FDF0272" Ref="#PWR0170"  Part="1"
+F 0 "#PWR0170" H 5500 2650 50  0001 C CNN
 F 1 "VBUS" H 5515 2973 50  0000 C CNN
 F 2 "" H 5500 2800 50  0001 C CNN
@@
 	9050 2800 9050 3300
 $Comp
-L Connector:TestPoint TP?
+L Connector:TestPoint TP11
 U 1 1 5FEB5241
 P 9700 2450
-F 0 "TP?" H 9758 2568 50  0000 L CNN
+F 0 "TP11" H 9758 2568 50  0000 L CNN
 F 1 "PROGVCC" H 9758 2477 50  0000 L CNN
-F 2 "" H 9900 2450 50  0001 C CNN
+F 2 "TestPoint:TestPoint_Pad_1.5x1.5mm" H 9900 2450 50  0001 C CNN
 F 3 "~" H 9900 2450 50  0001 C CNN
 	1    9700 2450
@@
 	9700 2800 10050 2800
 $Comp
-L Device:D_Schottky D?
+L Device:D_Schottky D12
 U 1 1 5FEB6937
 P 10200 2800
-F 0 "D?" H 10200 3016 50  0000 C CNN
+F 0 "D12" H 10200 3016 50  0000 C CNN
 F 1 "D_Schottky" H 10200 2925 50  0000 C CNN
-F 2 "" H 10200 2800 50  0001 C CNN
+F 2 "Diode_SMD:D_SOD-323" H 10200 2800 50  0001 C CNN
 F 3 "~" H 10200 2800 50  0001 C CNN
 	1    10200 2800
@@
 USB+
 $Comp
-L Connector:TestPoint TP?
+L Connector:TestPoint TP10
 U 1 1 60108CD6
 P 9600 4700
-F 0 "TP?" H 9658 4818 50  0000 L CNN
+F 0 "TP10" H 9658 4818 50  0000 L CNN
 F 1 "CH_BL_SEL" H 9658 4727 50  0000 L CNN
-F 2 "" H 9800 4700 50  0001 C CNN
+F 2 "TestPoint:TestPoint_Pad_1.5x1.5mm" H 9800 4700 50  0001 C CNN
 F 3 "~" H 9800 4700 50  0001 C CNN
 	1    9600 4700
