File: hardware/MeshangerV/input.sch (KiCad schematic (older format))
At the start: 26 parts

Commit message: more schematic
Parts:
- U?: symbol Useful_ICs:SN3218 -> MeshangerV-rescue:SN3218-Useful_ICs
- U?: symbol Useful_ICs:AT42QT2120 -> MeshangerV-rescue:AT42QT2120-Useful_ICs
Changed lines of the file:
@@
 EESchema Schematic File Version 4
 LIBS:MeshangerV-cache
-EELAYER 29 0
+EELAYER 26 0
 EELAYER END
 $Descr A4 11693 8268
 encoding utf-8
-Sheet 3 3
+Sheet 3 4
 Title ""
 Date ""
@@
 GND
 $Comp
-L Useful_ICs:SN3218 U?
+L MeshangerV-rescue:SN3218-Useful_ICs U?
 U 1 1 5FE09172
 P 2850 4250
@@
 $EndComp
 $Comp
-L Useful_ICs:AT42QT2120 U?
+L MeshangerV-rescue:AT42QT2120-Useful_ICs U?
 U 1 1 5FE0B088
 P 6750 1700

Commit message: schematic complete more or less
Parts:
- removed R? (x4): R_Small, symbol Device:R_Small
- added RN?: R_Pack04, symbol Device:R_Pack04
Connections:
- net +3V3: now also RN?.5 (R4.2), RN?.6 (R3.2), RN?.7 (R2.2), RN?.8 (R1.2)
- net INT: now also RN?.3 (R3.1)
- net LED_SD: now also RN?.4 (R4.1)
- net SCL: now also RN?.2 (R2.1)
- net SDA: now also RN?.1 (R1.1)
Changed lines of the file:
@@
 EESchema Schematic File Version 4
 LIBS:MeshangerV-cache
-EELAYER 26 0
+EELAYER 29 0
 EELAYER END
 $Descr A4 11693 8268
 encoding utf-8
-Sheet 3 4
+Sheet 3 5
 Title ""
 Date ""
@@
 GND
 $Comp
-L Device:R_Small R?
-U 1 1 5FEC910A
-P 1550 1850
-F 0 "R?" H 1609 1896 50  0000 L CNN
-F 1 "R_Small" H 1609 1805 50  0000 L CNN
-F 2 "" H 1550 1850 50  0001 C CNN
-F 3 "~" H 1550 1850 50  0001 C CNN
-	1    1550 1850
-	1    0    0    -1
-$EndComp
-$Comp
-L Device:R_Small R?
-U 1 1 5FEC96E3
-P 1150 1850
-F 0 "R?" H 1209 1896 50  0000 L CNN
-F 1 "R_Small" H 1209 1805 50  0000 L CNN
-F 2 "" H 1150 1850 50  0001 C CNN
-F 3 "~" H 1150 1850 50  0001 C CNN
-	1    1150 1850
-	1    0    0    -1
-$EndComp
-$Comp
 L power:+3V3 #PWR?
 U 1 1 5FEC9D64
@@
 Wire Wire Line
 	5700 800  5700 650
-$Comp
-L Device:R_Small R?
-U 1 1 5FED518F
-P 1900 1850
-F 0 "R?" H 1959 1896 50  0000 L CNN
-F 1 "R_Small" H 1959 1805 50  0000 L CNN
-F 2 "" H 1900 1850 50  0001 C CNN
-F 3 "~" H 1900 1850 50  0001 C CNN
-	1    1900 1850
-	1    0    0    -1
-$EndComp
 Wire Wire Line
 	1150 1750 1150 1550
 Wire Wire Line
-	1150 1550 1550 1550
-Wire Wire Line
-	1550 1550 1550 1750
+	1150 1550 1250 1550
+Wire Wire Line
+	1250 1550 1250 1750
 Connection ~ 1150 1550
 Wire Wire Line
 	1150 1550 1150 1450
 Wire Wire Line
-	1550 1550 1900 1550
-Wire Wire Line
-	1900 1550 1900 1750
-Connection ~ 1550 1550
-Wire Wire Line
-	1150 1950 1150 2150
-Wire Wire Line
-	1550 1950 1550 2150
-Wire Wire Line
-	1900 1950 1900 2150
-Text Label 1550 2150 0    50   ~ 0
+	1250 1550 1350 1550
+Wire Wire Line
+	1350 1550 1350 1750
+Connection ~ 1250 1550
+Text Label 1250 2400 1    50   ~ 0
 SCL
-Text Label 1900 2150 0    50   ~ 0
+Text Label 1350 2400 1    50   ~ 0
 T_INT
-Text Label 1150 2150 0    50   ~ 0
+Text Label 1150 2400 1    50   ~ 0
 SDA
 $Comp
@@
 Wire Wire Line
 	2000 1050 2300 1050
-$Comp
-L Device:R_Small R?
-U 1 1 5FF2D759
-P 2400 1850
-F 0 "R?" H 2459 1896 50  0000 L CNN
-F 1 "R_Small" H 2459 1805 50  0000 L CNN
-F 2 "" H 2400 1850 50  0001 C CNN
-F 3 "~" H 2400 1850 50  0001 C CNN
-	1    2400 1850
-	1    0    0    -1
-$EndComp
-Wire Wire Line
-	2400 1750 2400 1550
-Wire Wire Line
-	2400 1950 2400 2150
-Text Label 2400 2150 0    50   ~ 0
-GND
-Text Label 2400 1550 0    50   ~ 0
+Wire Wire Line
+	1450 1750 1450 1550
+Text Label 1450 2400 1    50   ~ 0
 LED_SD
+Wire Wire Line
+	1350 1550 1450 1550
+Connection ~ 1350 1550
+$Comp
+L Device:R_Pack04 RN?
+U 1 1 5FEA8355
+P 1350 1950
+AR Path="/5FEA8355" Ref="RN?"  Part="1"
+AR Path="/5FDFCE72/5FEA8355" Ref="RN?"  Part="1"
+F 0 "RN?" H 1538 1996 50  0000 L CNN
+F 1 "R_Pack04" H 1538 1905 50  0000 L CNN
+F 2 "" V 1625 1950 50  0001 C CNN
+F 3 "~" H 1350 1950 50  0001 C CNN
+	1    1350 1950
+	1    0    0    -1
+$EndComp
+Wire Wire Line
+	1150 2400 1150 2150
+Wire Wire Line
+	1250 2400 1250 2150
+Wire Wire Line
+	1350 2400 1350 2150
+Wire Wire Line
+	1450 2400 1450 2150
 $EndSCHEMATC

Commit message: routing has begun
Parts:
- C27, C28: renamed from C?; footprint (none) -> Capacitor_SMD:C_0603_1608Metric
- D10, D11, D6, D7, D8, D9: renamed from D?; footprint (none) -> LED_SMD:LED_Kingbright_APFA3010_3x1.5mm_Horizontal
- J4: renamed from J?; footprint (none) -> footprint:touchwheel
- R14, R15: renamed from R?; footprint (none) -> Resistor_SMD:R_0603_1608Metric
- RN2: renamed from RN?; footprint (none) -> Resistor_SMD:R_Array_Convex_4x0603
- TP1, TP2, TP3, TP4, TP5, TP6, TP7, TP8, TP9: renamed from TP?; footprint (none) -> TestPoint:TestPoint_Pad_4.0x4.0mm
- U7: renamed from U?; footprint Package_DFN_QFN:QFN-24-1EP_4x4mm_P0.5mm_EP2.65x2.65mm_ThermalVias -> Housings_DFN_QFN:QFN-24_4x4mm_Pitch0.5mm
- U8: renamed from U?; footprint Package_DFN_QFN:QFN-20-1EP_3x3mm_P0.45mm_EP1.6x1.6mm -> Housings_DFN_QFN:ST_UFQFPN-20_3x3mm_Pitch0.5mm
Connections:
- net 1B: now also U7.7 (LED01); no longer U7.9 (LED03)
- net 1R: now also U7.9 (LED03); no longer U7.7 (LED01)
- net 2B: now also U7.10 (LED04); no longer U7.12 (LED06)
- net 2R: now also U7.12 (LED06); no longer U7.10 (LED04)
- net 3B: now also U7.13 (LED07); no longer U7.15 (LED09)
- net 3R: now also U7.15 (LED09); no longer U7.13 (LED07)
- net 4B: now also U7.16 (LED10); no longer U7.18 (LED12)
- net 4R: now also U7.18 (LED12); no longer U7.16 (LED10)
- net 5B: now also U7.19 (LED13); no longer U7.21 (LED15)
- net 5R: now also U7.21 (LED15); no longer U7.19 (LED13)
- net 6B: now also U7.22 (LED16); no longer U7.1 (LED18)
- net 6R: now also U7.1 (LED18); no longer U7.22 (LED16)
